File: Power.kicad_sch (KiCad schematic)
At the start: 33 parts, among them J3 Conn_01x02, U2 TPS56121, U3 LD1117S33TR_SOT223

Commit message: Add part numbers for all capacitors
Parts:
- C10, C19, C20, C8, C9: Part No. (none) -> GRM32EC70J107ME15K
- C11: footprint Capacitor_SMD:C_1210_3225Metric -> Capacitor_SMD:C_0805_2012Metric; Part No. (none) -> GRM219R7YA105MA12D
- C12: Part No. (none) -> GRM21BR71C475ME51K
- C13: Part No. (none) -> GCM219R72A333KA37D
- C14, C4: Part No. (none) -> GCM21BR72A104KA37L
- C15: Part No. (none) -> CC0805KRX7R9BB391
- C16: Part No. (none) -> GRM21A5C2D120JW01D
- C17: Part No. (none) -> GRM21A5C2E821JWA1J
- C18: Part No. (none) -> GRM2165C2A102JA01D
- C21: footprint Capacitor_SMD:C_1210_3225Metric -> Capacitor_SMD:C_0805_2012Metric; Part No. CL32B105KBHNNNE -> GRM219R7YA105MA12D
- C22, C23, C24, C25: Part No. (none) -> GRM32ER71E226KE15K
- C3: Part No. (none) -> GRM21BR61C106KE15K
Changed lines of the file:
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@@
+      (effects (font (size 1.27 1.27)) hide)
+    )
+    (property "Part No." "GRM32ER71E226KE15K" (at 174.625 81.28 0)
       (effects (font (size 1.27 1.27)) hide)
     )
@@
     )
     (property "Description" "" (at 201.295 81.28 0)
+      (effects (font (size 1.27 1.27)) hide)
+    )
+    (property "Part No." "GRM32ER71E226KE15K" (at 201.295 81.28 0)
       (effects (font (size 1.27 1.27)) hide)
     )
@@
       (effects (font (size 1.27 1.27)) hide)
     )
+    (property "Part No." "GRM21A5C2D120JW01D" (at 64.77 153.67 0)
+      (effects (font (size 1.27 1.27)) hide)
+    )
     (pin "1")
     (pin "2")
@@
       (effects (font (size 1.27 1.27)) hide)
     )
-    (property "Part No." "" (at 35.56 90.805 0)
+    (property "Part No." "GCM219R72A333KA37D" (at 35.56 90.805 0)
       (effects (font (size 1.27 1.27)) hide)
     )
@@
       (effects (font (size 1.27 1.27)) hide)
     )
+    (property "Part No." "GCM21BR72A104KA37L" (at 54.61 33.02 0)
+      (effects (font (size 1.27 1.27)) hide)
+    )
     (pin "1")
     (pin "2")
@@
       (effects (font (size 1.27 1.27)) hide)
     )
+    (property "Part No." "GRM32EC70J107ME15K" (at 187.96 106.045 0)
+      (effects (font (size 1.27 1.27)) hide)
+    )
     (pin "1")
     (pin "2")
@@
       (effects (font (size 1.27 1.27)) hide)
     )
-    (property "Part No." "" (at 110.49 153.67 0)
+    (property "Part No." "GRM21A5C2E821JWA1J" (at 110.49 153.67 0)
       (effects (font (size 1.27 1.27)) hide)
     )
@@
       (effects (font (size 1.27 1.27)) hide)
     )
-    (property "Part No." "" (at 90.17 33.02 0)
+    (property "Part No." "GRM21BR61C106KE15K" (at 90.17 33.02 0)
       (effects (font (size 1.27 1.27)) hide)
     )
@@
       (effects (font (size 1.27 1.27)) hide)
     )
+    (property "Part No." "GRM32EC70J107ME15K" (at 174.625 106.045 0)
+      (effects (font (size 1.27 1.27)) hide)
+    )
     (pin "1")
     (pin "2")
@@
     )
     (property "Description" "Capacitor, Ceramic, 50 V, X7R, 10%" (at 59.69 143.51 0)
+      (effects (font (size 1.27 1.27)) hide)
+    )
+    (property "Part No." "CC0805KRX7R9BB391" (at 59.69 143.51 0)
       (effects (font (size 1.27 1.27)) hide)
     )
@@
       (effects (font (size 1.27 1.27)) (justify left))
     )
-    (property "Footprint" "Capacitor_SMD:C_1210_3225Metric" (at 162.2552 85.09 0)
+    (property "Footprint" "Capacitor_SMD:C_0805_2012Metric" (at 162.2552 85.09 0)
       (effects (font (size 1.27 1.27)) hide)
     )
@@
       (effects (font (size 1.27 1.27)) hide)
     )
-    (property "Part No." "CL32B105KBHNNNE" (at 161.29 81.28 0)
+    (property "Part No." "GRM219R7YA105MA12D" (at 161.29 81.28 0)
       (effects (font (size 1.27 1.27)) hide)
     )
@@
       (effects (font (size 1.27 1.27)) hide)
     )
+    (property "Part No." "GRM32EC70J107ME15K" (at 201.295 106.045 0)
+      (effects (font (size 1.27 1.27)) hide)
+    )
     (pin "1")
     (pin "2")
@@
       (effects (font (size 1.27 1.27)) hide)
     )
+    (property "Part No." "GRM32EC70J107ME15K" (at 214.63 106.045 0)
+      (effects (font (size 1.27 1.27)) hide)
+    )
     (pin "1")
     (pin "2")
@@
       (effects (font (size 1.27 1.27)) (justify left))
     )
-    (property "Footprint" "Capacitor_SMD:C_1210_3225Metric" (at 68.2752 70.485 0)
+    (property "Footprint" "Capacitor_SMD:C_0805_2012Metric" (at 68.2752 70.485 0)
       (effects (font (size 1.27 1.27)) hide)
     )
@@
       (effects (font (size 1.27 1.27)) hide)
     )
-    (property "Part No." "" (at 67.31 66.675 0)
+    (property "Part No." "GRM219R7YA105MA12D" (at 67.31 66.675 0)
       (effects (font (size 1.27 1.27)) hide)
     )
@@
       (effects (font (size 1.27 1.27)) hide)
     )
-    (property "Part No." "" (at 161.29 106.045 0)
+    (property "Part No." "GRM32EC70J107ME15K" (at 161.29 106.045 0)
       (effects (font (size 1.27 1.27)) hide)
     )
@@
       (effects (font (size 1.27 1.27)) hide)
     )
+    (property "Part No." "GRM32ER71E226KE15K" (at 214.63 81.28 0)
+      (effects (font (size 1.27 1.27)) hide)
+    )
     (pin "1")
     (pin "2")
@@
       (effects (font (size 1.27 1.27)) hide)
     )
+    (property "Part No." "GRM32ER71E226KE15K" (at 187.96 81.28 0)
+      (effects (font (size 1.27 1.27)) hide)
+    )
     (pin "1")
     (pin "2")
@@
       (effects (font (size 1.27 1.27)) hide)
     )
-    (property "Part No." "" (at 116.84 124.46 0)
+    (property "Part No." "GRM2165C2A102JA01D" (at 116.84 124.46 0)
       (effects (font (size 1.27 1.27)) hide)
     )
@@
       (effects (font (size 1.27 1.27)) hide)
     )
-    (property "Part No." "" (at 85.725 124.46 0)
+    (property "Part No." "GCM21BR72A104KA37L" (at 85.725 124.46 0)
       (effects (font (size 1.27 1.27)) hide)
     )
@@
       (effects (font (size 1.27 1.27)) hide)
     )
-    (property "Part No." "" (at 80.01 66.675 0)
-      (effects (font (size 1.27 1.27)) hide)
-    )
+    (property "Part No." "GRM21BR71C475ME51K" (at 80.01 66.675 0)
+      (effects (font (size 1.27 1.27)) hide)
+    )

Commit message: Adjust layout
Parts:
- U2: footprint Package_DFN_QFN:DFN-22-1EP_5x6mm_P0.5mm_EP3.14x4.3mm -> Marks_Footprints:DFN-22-1EP_5x6mm_P0.5mm_EP3.14x4.3mm
Changed lines of the file:
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@@
       (effects (font (size 1.27 1.27)) (justify left))
     )
-    (property "Footprint" "Package_DFN_QFN:DFN-22-1EP_5x6mm_P0.5mm_EP3.14x4.3mm" (at 59.69 113.03 0)
+    (property "Footprint" "Marks_Footprints:DFN-22-1EP_5x6mm_P0.5mm_EP3.14x4.3mm" (at 59.69 113.03 0)
       (effects (font (size 1.27 1.27)) hide)
     )

Commit message: Adjust buck converter thermal vias
Parts:
- R1: Part No. (none) -> RC0805FR-071K78L
- R2: Part No. (none) -> RC0805FR-075R1L
- R3: Part No. (none) -> RC0805FR-07442KL
- R4: Part No. (none) -> RC0805FR-07200KL
- R5: Part No. (none) -> RC0805FR-0749R9L
- R6: Part No. (none) -> RC0805FR-076K2L
- R7: Part No. (none) -> RC0805FR-0722KL
- R9: Part No. (none) -> RC0805FR-101RL
- U3: Part No. (none) -> LD1117S33TR
Changed lines of the file:
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@@
       (effects (font (size 1.27 1.27)) hide)
     )
-    (property "Part No." "" (at 73.66 120.65 0)
+    (property "Part No." "RC0805FR-075R1L" (at 73.66 120.65 0)
       (effects (font (size 1.27 1.27)) hide)
     )
@@
       (effects (font (size 1.27 1.27)) hide)
     )
+    (property "Part No." "RC0805FR-071K78L" (at 92.075 66.675 0)
+      (effects (font (size 1.27 1.27)) hide)
+    )
     (pin "1")
     (pin "2")
@@
       (effects (font (size 1.27 1.27)) hide)
     )
+    (property "Part No." "RC0805FR-07442KL" (at 69.85 143.51 0)
+      (effects (font (size 1.27 1.27)) hide)
+    )
     (pin "1")
     (pin "2")
@@
       (effects (font (size 1.27 1.27)) hide)
     )
-    (property "Part No." "" (at 73.025 26.67 0)
+    (property "Part No." "LD1117S33TR" (at 73.025 26.67 0)
       (effects (font (size 1.27 1.27)) hide)
     )
@@
       (effects (font (size 1.27 1.27)) hide)
     )
-    (property "Part No." "" (at 103.505 120.015 0)
+    (property "Part No." "RC0805FR-101RL" (at 103.505 120.015 0)
       (effects (font (size 1.27 1.27)) hide)
     )
@@
       (effects (font (size 1.27 1.27)) hide)
     )
-    (property "Part No." "" (at 83.185 153.67 0)
+    (property "Part No." "RC0805FR-0722KL" (at 83.185 153.67 0)
       (effects (font (size 1.27 1.27)) hide)
     )
@@
       (effects (font (size 1.27 1.27)) hide)
     )
+    (property "Part No." "RC0805FR-076K2L" (at 97.79 153.67 0)
+      (effects (font (size 1.27 1.27)) hide)
+    )
     (pin "1")
     (pin "2")
@@
       (effects (font (size 1.27 1.27)) hide)
     )
+    (property "Part No." "RC0805FR-0749R9L" (at 123.19 143.51 0)
+      (effects (font (size 1.27 1.27)) hide)
+    )
     (pin "1")
     (pin "2")
@@
       (effects (font (size 1.27 1.27)) hide)
     )
-    (property "Part No." "" (at 101.6 143.51 0)
-      (effects (font (size 1.27 1.27)) hide)
-    )
+    (property "Part No." "RC0805FR-07200KL" (at 101.6 143.51 0)
+      (effects (font (size 1.27 1.27)) hide)
+    )
